File: CAD/KiCAD/digitizer/digitizer.kicad_pcb (KiCad board)
At the start: 2 copper layers, 254 x 254 mm, 77 parts, among them J1 Conn_01x06, J1_01 Conn_02x40_Odd_Even, J1_02 Conn_02x40_Odd_Even, J1_03 Conn_02x40_Odd_Even, J1_04 Conn_02x40_Odd_Even, J1_05 Conn_02x40_Odd_Even, J1_06 Conn_02x40_Odd_Even, J1_07 Conn_02x40_Odd_Even, J1_08 Conn_02x40_Odd_Even, J1_09 Conn_02x40_Odd_Even, J1_10 Conn_02x40_Odd_Even, J1_11 Conn_02x40_Odd_Even, J1_12 Conn_02x40_Odd_Even, J1_13 Conn_02x40_Odd_Even, J1_14 Conn_02x40_Odd_Even, J1_15 Conn_02x40_Odd_Even, J1_16 Conn_02x40_Odd_Even, J1_17 Conn_02x40_Odd_Even, J1_18 Conn_02x40_Odd_Even, J1_19 Conn_02x40_Odd_Even, J1_20 Conn_02x40_Odd_Even, J1_21 Conn_02x40_Odd_Even, J1_22 Conn_02x40_Odd_Even, J1_23 Conn_02x40_Odd_Even, J1_24 Conn_02x40_Odd_Even, J1_25 Conn_02x40_Odd_Even, J1_26 Conn_02x40_Odd_Even, J1_27 Conn_02x40_Odd_Even, J1_28 Conn_02x40_Odd_Even, J1_29 Conn_02x40_Odd_Even, J1_30 Conn_02x40_Odd_Even, J1_31 Conn_02x40_Odd_Even, J1_32 Conn_02x40_Odd_Even, J2_01 Conn_02x24_Odd_Even, J2_02 Conn_02x24_Odd_Even, J2_03 Conn_02x24_Odd_Even, J2_04 Conn_02x24_Odd_Even, J2_05 Conn_02x24_Odd_Even, J2_06 Conn_02x24_Odd_Even, J2_07 Conn_02x24_Odd_Even, J2_08 Conn_02x24_Odd_Even, J2_09 Conn_02x24_Odd_Even, J2_10 Conn_02x24_Odd_Even, J2_11 Conn_02x24_Odd_Even, J2_12 Conn_02x24_Odd_Even, J2_13 Conn_02x24_Odd_Even, J2_14 Conn_02x24_Odd_Even, J2_15 Conn_02x24_Odd_Even, J2_16 Conn_02x24_Odd_Even, J2_17 Conn_02x24_Odd_Even, J2_18 Conn_02x24_Odd_Even, J2_19 Conn_02x24_Odd_Even, J2_20 Conn_02x24_Odd_Even, J2_21 Conn_02x24_Odd_Even, J2_22 Conn_02x24_Odd_Even, J2_23 Conn_02x24_Odd_Even, J2_24 Conn_02x24_Odd_Even, J2_25 Conn_02x24_Odd_Even, J2_26 Conn_02x24_Odd_Even, J2_27 Conn_02x24_Odd_Even, J2_28 Conn_02x24_Odd_Even, J2_29 Conn_02x24_Odd_Even, J2_30 Conn_02x24_Odd_Even, J2_31 Conn_02x24_Odd_Even, J2_32 Conn_02x24_Odd_Even, P1_1 Conn_01x06, P1_2 Conn_01x06, P1_3 Conn_01x06, P1_4 Conn_01x06, P3_1 Conn_01x10, P3_2 Conn_01x10, P3_3 Conn_01x10, P3_4 Conn_01x10, P4_1 Conn_01x10, P4_2 Conn_01x10, P4_3 Conn_01x10, P4_4 Conn_01x10

Commit message: wip
Parts:
- added J2: Conn_01x06, Connector_PinHeader_2.54mm:PinHeader_1x06_P2.54mm_Vertical, F.Cu at (53.3, 257.3)
- added R1: 10k, Resistor_THT:R_Axial_DIN0207_L6.3mm_D2.5mm_P15.24mm_Horizontal, F.Cu at (76.5, 178.6)
- added R2: 10k, Resistor_THT:R_Axial_DIN0207_L6.3mm_D2.5mm_P15.24mm_Horizontal, F.Cu at (76.2, 183.6)
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Connections:
- J1_01 pad 10: R3 -> R30
- J1_01 pad 11: R3 -> R30
- J1_01 pad 14: R4 -> R29
- J1_01 pad 15: R4 -> R29
- J1_01 pad 18: R5 -> R28
- J1_01 pad 19: R5 -> R28
- J1_01 pad 2: R1 -> R32
- J1_01 pad 22: R6 -> R27
- J1_01 pad 23: R6 -> R27
- J1_01 pad 26: R7 -> R26
- J1_01 pad 27: R7 -> R26
- J1_01 pad 3: R1 -> R32
- J1_01 pad 30: R8 -> R25
- J1_01 pad 31: R8 -> R25
- J1_01 pad 34: R9 -> R24
- J1_01 pad 35: R9 -> R24
- J1_01 pad 38: R10 -> R23
- J1_01 pad 39: R10 -> R23
- J1_01 pad 42: R11 -> R22
- J1_01 pad 43: R11 -> R22
- J1_01 pad 46: R12 -> R21
- J1_01 pad 47: R12 -> R21
- J1_01 pad 50: R13 -> R20
- J1_01 pad 51: R13 -> R20
- J1_01 pad 54: R14 -> R19
- J1_01 pad 55: R14 -> R19
- J1_01 pad 58: R15 -> R18
- J1_01 pad 59: R15 -> R18
- J1_01 pad 6: R2 -> R31
- J1_01 pad 62: R16 -> R17
- J1_01 pad 63: R16 -> R17
- J1_01 pad 66: R17 -> R16
- J1_01 pad 67: R17 -> R16
- J1_01 pad 7: R2 -> R31
- J1_01 pad 70: R18 -> R15
- J1_01 pad 71: R18 -> R15
- J1_01 pad 74: R19 -> R14
- J1_01 pad 75: R19 -> R14
- J1_01 pad 78: R20 -> R13
- J1_01 pad 79: R20 -> R13
- J1_02 pad 10: R3 -> R30
- J1_02 pad 11: R3 -> R30
- J1_02 pad 14: R4 -> R29
- J1_02 pad 15: R4 -> R29
- J1_02 pad 18: R5 -> R28
- J1_02 pad 19: R5 -> R28
- J1_02 pad 2: R1 -> R32
- J1_02 pad 22: R6 -> R27
- J1_02 pad 23: R6 -> R27
- J1_02 pad 26: R7 -> R26
- J1_02 pad 27: R7 -> R26
- J1_02 pad 3: R1 -> R32
- J1_02 pad 30: R8 -> R25
- J1_02 pad 31: R8 -> R25
- J1_02 pad 34: R9 -> R24
- J1_02 pad 35: R9 -> R24
- J1_02 pad 38: R10 -> R23
- J1_02 pad 39: R10 -> R23
- J1_02 pad 42: R11 -> R22
- J1_02 pad 43: R11 -> R22
- J1_02 pad 46: R12 -> R21
- J1_02 pad 47: R12 -> R21
- J1_02 pad 50: R13 -> R20
- J1_02 pad 51: R13 -> R20
- J1_02 pad 54: R14 -> R19
- J1_02 pad 55: R14 -> R19
- J1_02 pad 58: R15 -> R18
- J1_02 pad 59: R15 -> R18
- J1_02 pad 6: R2 -> R31
- J1_02 pad 62: R16 -> R17
- J1_02 pad 63: R16 -> R17
- J1_02 pad 66: R17 -> R16
- J1_02 pad 67: R17 -> R16
- J1_02 pad 7: R2 -> R31
- J1_02 pad 70: R18 -> R15
- J1_02 pad 71: R18 -> R15
- J1_02 pad 74: R19 -> R14
- J1_02 pad 75: R19 -> R14
- J1_02 pad 78: R20 -> R13
- J1_02 pad 79: R20 -> R13
- J1_03 pad 10: R3 -> R30
- J1_03 pad 11: R3 -> R30
- J1_03 pad 14: R4 -> R29
- J1_03 pad 15: R4 -> R29
- J1_03 pad 18: R5 -> R28
- J1_03 pad 19: R5 -> R28
- J1_03 pad 2: R1 -> R32
- J1_03 pad 22: R6 -> R27
- J1_03 pad 23: R6 -> R27
- J1_03 pad 26: R7 -> R26
- J1_03 pad 27: R7 -> R26
- J1_03 pad 3: R1 -> R32
- J1_03 pad 30: R8 -> R25
- J1_03 pad 31: R8 -> R25
- J1_03 pad 34: R9 -> R24
- J1_03 pad 35: R9 -> R24
- J1_03 pad 38: R10 -> R23
- J1_03 pad 39: R10 -> R23
- J1_03 pad 42: R11 -> R22
- J1_03 pad 43: R11 -> R22
- J1_03 pad 46: R12 -> R21
- J1_03 pad 47: R12 -> R21
- J1_03 pad 50: R13 -> R20
- J1_03 pad 51: R13 -> R20
- J1_03 pad 54: R14 -> R19
- J1_03 pad 55: R14 -> R19
- J1_03 pad 58: R15 -> R18
- J1_03 pad 59: R15 -> R18
- J1_03 pad 6: R2 -> R31
- J1_03 pad 62: R16 -> R17
- J1_03 pad 63: R16 -> R17
- J1_03 pad 66: R17 -> R16
- J1_03 pad 67: R17 -> R16
- J1_03 pad 7: R2 -> R31
- J1_03 pad 70: R18 -> R15
- J1_03 pad 71: R18 -> R15
- J1_03 pad 74: R19 -> R14
- J1_03 pad 75: R19 -> R14
- J1_03 pad 78: R20 -> R13
- J1_03 pad 79: R20 -> R13
- J1_04 pad 10: R3 -> R30
- J1_04 pad 11: R3 -> R30
- J1_04 pad 14: R4 -> R29
- J1_04 pad 15: R4 -> R29
- J1_04 pad 18: R5 -> R28
- J1_04 pad 19: R5 -> R28
- J1_04 pad 2: R1 -> R32
- J1_04 pad 22: R6 -> R27
- J1_04 pad 23: R6 -> R27
- J1_04 pad 26: R7 -> R26
- J1_04 pad 27: R7 -> R26
- J1_04 pad 3: R1 -> R32
- J1_04 pad 30: R8 -> R25
- J1_04 pad 31: R8 -> R25
- J1_04 pad 34: R9 -> R24
- J1_04 pad 35: R9 -> R24
- J1_04 pad 38: R10 -> R23
- J1_04 pad 39: R10 -> R23
- J1_04 pad 42: R11 -> R22
- J1_04 pad 43: R11 -> R22
- J1_04 pad 46: R12 -> R21
- J1_04 pad 47: R12 -> R21
- J1_04 pad 50: R13 -> R20
- J1_04 pad 51: R13 -> R20
- J1_04 pad 54: R14 -> R19
- J1_04 pad 55: R14 -> R19
- J1_04 pad 58: R15 -> R18
- J1_04 pad 59: R15 -> R18
- J1_04 pad 6: R2 -> R31
- J1_04 pad 62: R16 -> R17
- J1_04 pad 63: R16 -> R17
- J1_04 pad 66: R17 -> R16
- J1_04 pad 67: R17 -> R16
- J1_04 pad 7: R2 -> R31
- J1_04 pad 70: R18 -> R15
- J1_04 pad 71: R18 -> R15
- J1_04 pad 74: R19 -> R14
- J1_04 pad 75: R19 -> R14
- J1_04 pad 78: R20 -> R13
- J1_04 pad 79: R20 -> R13
- J1_05 pad 10: R3 -> R30
- J1_05 pad 11: R3 -> R30
- J1_05 pad 14: R4 -> R29
- J1_05 pad 15: R4 -> R29
- J1_05 pad 18: R5 -> R28
- J1_05 pad 19: R5 -> R28
- J1_05 pad 2: R1 -> R32
- J1_05 pad 22: R6 -> R27
- J1_05 pad 23: R6 -> R27
- J1_05 pad 26: R7 -> R26
- J1_05 pad 27: R7 -> R26
- J1_05 pad 3: R1 -> R32
- J1_05 pad 30: R8 -> R25
- J1_05 pad 31: R8 -> R25
- J1_05 pad 34: R9 -> R24
- J1_05 pad 35: R9 -> R24
- J1_05 pad 38: R10 -> R23
- J1_05 pad 39: R10 -> R23
- J1_05 pad 42: R11 -> R22
- J1_05 pad 43: R11 -> R22
- J1_05 pad 46: R12 -> R21
- J1_05 pad 47: R12 -> R21
- J1_05 pad 50: R13 -> R20
- J1_05 pad 51: R13 -> R20
- J1_05 pad 54: R14 -> R19
- J1_05 pad 55: R14 -> R19
- J1_05 pad 58: R15 -> R18
- J1_05 pad 59: R15 -> R18
- J1_05 pad 6: R2 -> R31
- J1_05 pad 62: R16 -> R17
- J1_05 pad 63: R16 -> R17
- J1_05 pad 66: R17 -> R16
- J1_05 pad 67: R17 -> R16
- J1_05 pad 7: R2 -> R31
- J1_05 pad 70: R18 -> R15
- J1_05 pad 71: R18 -> R15
- J1_05 pad 74: R19 -> R14
- J1_05 pad 75: R19 -> R14
- J1_05 pad 78: R20 -> R13
- J1_05 pad 79: R20 -> R13
- J1_06 pad 10: R3 -> R30
- J1_06 pad 11: R3 -> R30
- J1_06 pad 14: R4 -> R29
- J1_06 pad 15: R4 -> R29
- J1_06 pad 18: R5 -> R28
- J1_06 pad 19: R5 -> R28
- J1_06 pad 2: R1 -> R32
- J1_06 pad 22: R6 -> R27
- J1_06 pad 23: R6 -> R27
- J1_06 pad 26: R7 -> R26
- J1_06 pad 27: R7 -> R26
- J1_06 pad 3: R1 -> R32
- J1_06 pad 30: R8 -> R25
- J1_06 pad 31: R8 -> R25
- J1_06 pad 34: R9 -> R24
- J1_06 pad 35: R9 -> R24
- J1_06 pad 38: R10 -> R23
- J1_06 pad 39: R10 -> R23
- J1_06 pad 42: R11 -> R22
- J1_06 pad 43: R11 -> R22
- J1_06 pad 46: R12 -> R21
- J1_06 pad 47: R12 -> R21
- J1_06 pad 50: R13 -> R20
- J1_06 pad 51: R13 -> R20
- J1_06 pad 54: R14 -> R19
- J1_06 pad 55: R14 -> R19
- J1_06 pad 58: R15 -> R18
- J1_06 pad 59: R15 -> R18
- J1_06 pad 6: R2 -> R31
- J1_06 pad 62: R16 -> R17
- J1_06 pad 63: R16 -> R17
- J1_06 pad 66: R17 -> R16
- J1_06 pad 67: R17 -> R16
- J1_06 pad 7: R2 -> R31
- J1_06 pad 70: R18 -> R15
- J1_06 pad 71: R18 -> R15
- J1_06 pad 74: R19 -> R14
- J1_06 pad 75: R19 -> R14
- J1_06 pad 78: R20 -> R13
- J1_06 pad 79: R20 -> R13
- J1_07 pad 10: R3 -> R30
- J1_07 pad 11: R3 -> R30
- J1_07 pad 14: R4 -> R29
- J1_07 pad 15: R4 -> R29
- J1_07 pad 18: R5 -> R28
- J1_07 pad 19: R5 -> R28
- J1_07 pad 2: R1 -> R32
- J1_07 pad 22: R6 -> R27
- J1_07 pad 23: R6 -> R27
- J1_07 pad 26: R7 -> R26
- J1_07 pad 27: R7 -> R26
- J1_07 pad 3: R1 -> R32
- J1_07 pad 30: R8 -> R25
- J1_07 pad 31: R8 -> R25
- J1_07 pad 34: R9 -> R24
- J1_07 pad 35: R9 -> R24
- J1_07 pad 38: R10 -> R23
- J1_07 pad 39: R10 -> R23
- J1_07 pad 42: R11 -> R22
- J1_07 pad 43: R11 -> R22
- J1_07 pad 46: R12 -> R21
- J1_07 pad 47: R12 -> R21
- J1_07 pad 50: R13 -> R20
- J1_07 pad 51: R13 -> R20
- J1_07 pad 54: R14 -> R19
- J1_07 pad 55: R14 -> R19
- J1_07 pad 58: R15 -> R18
- J1_07 pad 59: R15 -> R18
- J1_07 pad 6: R2 -> R31
- J1_07 pad 62: R16 -> R17
- J1_07 pad 63: R16 -> R17
- J1_07 pad 66: R17 -> R16
- J1_07 pad 67: R17 -> R16
- J1_07 pad 7: R2 -> R31
- J1_07 pad 70: R18 -> R15
- J1_07 pad 71: R18 -> R15
- J1_07 pad 74: R19 -> R14
- J1_07 pad 75: R19 -> R14
- J1_07 pad 78: R20 -> R13
- J1_07 pad 79: R20 -> R13
- J1_08 pad 10: R3 -> R30
- J1_08 pad 11: R3 -> R30
- J1_08 pad 14: R4 -> R29
- J1_08 pad 15: R4 -> R29
- J1_08 pad 18: R5 -> R28
- J1_08 pad 19: R5 -> R28
- J1_08 pad 2: R1 -> R32
- J1_08 pad 22: R6 -> R27
- J1_08 pad 23: R6 -> R27
- J1_08 pad 26: R7 -> R26
- J1_08 pad 27: R7 -> R26
- J1_08 pad 3: R1 -> R32
- J1_08 pad 30: R8 -> R25
- J1_08 pad 31: R8 -> R25
- J1_08 pad 34: R9 -> R24
- J1_08 pad 35: R9 -> R24
- J1_08 pad 38: R10 -> R23
- J1_08 pad 39: R10 -> R23
- J1_08 pad 42: R11 -> R22
- J1_08 pad 43: R11 -> R22
- J1_08 pad 46: R12 -> R21
- J1_08 pad 47: R12 -> R21
- J1_08 pad 50: R13 -> R20
- J1_08 pad 51: R13 -> R20
- J1_08 pad 54: R14 -> R19
- J1_08 pad 55: R14 -> R19
- J1_08 pad 58: R15 -> R18
- J1_08 pad 59: R15 -> R18
- J1_08 pad 6: R2 -> R31
- J1_08 pad 62: R16 -> R17
- J1_08 pad 63: R16 -> R17
- J1_08 pad 66: R17 -> R16
- J1_08 pad 67: R17 -> R16
- J1_08 pad 7: R2 -> R31
- J1_08 pad 70: R18 -> R15
- J1_08 pad 71: R18 -> R15
- J1_08 pad 74: R19 -> R14
- J1_08 pad 75: R19 -> R14
- J1_08 pad 78: R20 -> R13
- J1_08 pad 79: R20 -> R13
- J1_09 pad 10: R3 -> R30
- J1_09 pad 11: R3 -> R30
- J1_09 pad 14: R4 -> R29
- J1_09 pad 15: R4 -> R29
- J1_09 pad 18: R5 -> R28
- J1_09 pad 19: R5 -> R28
- J1_09 pad 2: R1 -> R32
- J1_09 pad 22: R6 -> R27
- J1_09 pad 23: R6 -> R27
- J1_09 pad 26: R7 -> R26
- J1_09 pad 27: R7 -> R26
- J1_09 pad 3: R1 -> R32
- J1_09 pad 30: R8 -> R25
- J1_09 pad 31: R8 -> R25
- J1_09 pad 34: R9 -> R24
- J1_09 pad 35: R9 -> R24
- J1_09 pad 38: R10 -> R23
- J1_09 pad 39: R10 -> R23
- J1_09 pad 42: R11 -> R22
- J1_09 pad 43: R11 -> R22
- J1_09 pad 46: R12 -> R21
- J1_09 pad 47: R12 -> R21
- J1_09 pad 50: R13 -> R20
- J1_09 pad 51: R13 -> R20
- J1_09 pad 54: R14 -> R19
- J1_09 pad 55: R14 -> R19
- J1_09 pad 58: R15 -> R18
- J1_09 pad 59: R15 -> R18
- J1_09 pad 6: R2 -> R31
- J1_09 pad 62: R16 -> R17
- J1_09 pad 63: R16 -> R17
- J1_09 pad 66: R17 -> R16
- J1_09 pad 67: R17 -> R16
- J1_09 pad 7: R2 -> R31
- J1_09 pad 70: R18 -> R15
- J1_09 pad 71: R18 -> R15
- J1_09 pad 74: R19 -> R14
- J1_09 pad 75: R19 -> R14
- J1_09 pad 78: R20 -> R13
- J1_09 pad 79: R20 -> R13
- J1_10 pad 10: R3 -> R30
- J1_10 pad 11: R3 -> R30
- J1_10 pad 14: R4 -> R29
- J1_10 pad 15: R4 -> R29
- J1_10 pad 18: R5 -> R28
- J1_10 pad 19: R5 -> R28
- J1_10 pad 2: R1 -> R32
- J1_10 pad 22: R6 -> R27
- J1_10 pad 23: R6 -> R27
- J1_10 pad 26: R7 -> R26
- J1_10 pad 27: R7 -> R26
- J1_10 pad 3: R1 -> R32
- J1_10 pad 30: R8 -> R25
- J1_10 pad 31: R8 -> R25
- J1_10 pad 34: R9 -> R24
- J1_10 pad 35: R9 -> R24
- J1_10 pad 38: R10 -> R23
- J1_10 pad 39: R10 -> R23
- J1_10 pad 42: R11 -> R22
- J1_10 pad 43: R11 -> R22
- J1_10 pad 46: R12 -> R21
- J1_10 pad 47: R12 -> R21
- J1_10 pad 50: R13 -> R20
- J1_10 pad 51: R13 -> R20
- J1_10 pad 54: R14 -> R19
- J1_10 pad 55: R14 -> R19
- J1_10 pad 58: R15 -> R18
- J1_10 pad 59: R15 -> R18
- J1_10 pad 6: R2 -> R31
- J1_10 pad 62: R16 -> R17
- J1_10 pad 63: R16 -> R17
- J1_10 pad 66: R17 -> R16
- J1_10 pad 67: R17 -> R16
- J1_10 pad 7: R2 -> R31
- J1_10 pad 70: R18 -> R15
- J1_10 pad 71: R18 -> R15
- J1_10 pad 74: R19 -> R14
- J1_10 pad 75: R19 -> R14
- J1_10 pad 78: R20 -> R13
- J1_10 pad 79: R20 -> R13
- J1_11 pad 10: R3 -> R30
- J1_11 pad 11: R3 -> R30
- J1_11 pad 14: R4 -> R29
- J1_11 pad 15: R4 -> R29
- J1_11 pad 18: R5 -> R28
- J1_11 pad 19: R5 -> R28
- J1_11 pad 2: R1 -> R32
- J1_11 pad 22: R6 -> R27
- J1_11 pad 23: R6 -> R27
- J1_11 pad 26: R7 -> R26
- J1_11 pad 27: R7 -> R26
- J1_11 pad 3: R1 -> R32
- J1_11 pad 30: R8 -> R25
- J1_11 pad 31: R8 -> R25
- J1_11 pad 34: R9 -> R24
- J1_11 pad 35: R9 -> R24
- J1_11 pad 38: R10 -> R23
- J1_11 pad 39: R10 -> R23
- J1_11 pad 42: R11 -> R22
- J1_11 pad 43: R11 -> R22
- J1_11 pad 46: R12 -> R21
- J1_11 pad 47: R12 -> R21
- J1_11 pad 50: R13 -> R20
- J1_11 pad 51: R13 -> R20
- J1_11 pad 54: R14 -> R19
- J1_11 pad 55: R14 -> R19
- J1_11 pad 58: R15 -> R18
- J1_11 pad 59: R15 -> R18
- J1_11 pad 6: R2 -> R31
- J1_11 pad 62: R16 -> R17
- J1_11 pad 63: R16 -> R17
- J1_11 pad 66: R17 -> R16
- J1_11 pad 67: R17 -> R16
- J1_11 pad 7: R2 -> R31
- J1_11 pad 70: R18 -> R15
- J1_11 pad 71: R18 -> R15
- J1_11 pad 74: R19 -> R14
- J1_11 pad 75: R19 -> R14
- J1_11 pad 78: R20 -> R13
- J1_11 pad 79: R20 -> R13
- J1_12 pad 10: R3 -> R30
- J1_12 pad 11: R3 -> R30
- J1_12 pad 14: R4 -> R29
- J1_12 pad 15: R4 -> R29
- J1_12 pad 18: R5 -> R28
- J1_12 pad 19: R5 -> R28
- J1_12 pad 2: R1 -> R32
- J1_12 pad 22: R6 -> R27
- J1_12 pad 23: R6 -> R27
- J1_12 pad 26: R7 -> R26
- J1_12 pad 27: R7 -> R26
- J1_12 pad 3: R1 -> R32
- J1_12 pad 30: R8 -> R25
- J1_12 pad 31: R8 -> R25
- J1_12 pad 34: R9 -> R24
- J1_12 pad 35: R9 -> R24
- J1_12 pad 38: R10 -> R23
- J1_12 pad 39: R10 -> R23
- J1_12 pad 42: R11 -> R22
- J1_12 pad 43: R11 -> R22
- J1_12 pad 46: R12 -> R21
- J1_12 pad 47: R12 -> R21
- J1_12 pad 50: R13 -> R20
- J1_12 pad 51: R13 -> R20
- J1_12 pad 54: R14 -> R19
- J1_12 pad 55: R14 -> R19
- J1_12 pad 58: R15 -> R18
- J1_12 pad 59: R15 -> R18
- J1_12 pad 6: R2 -> R31
- J1_12 pad 62: R16 -> R17
- J1_12 pad 63: R16 -> R17
- J1_12 pad 66: R17 -> R16
- J1_12 pad 67: R17 -> R16
- J1_12 pad 7: R2 -> R31
- J1_12 pad 70: R18 -> R15
- J1_12 pad 71: R18 -> R15
- J1_12 pad 74: R19 -> R14
- J1_12 pad 75: R19 -> R14
- J1_12 pad 78: R20 -> R13
- J1_12 pad 79: R20 -> R13
- J1_13 pad 10: R3 -> R30
- J1_13 pad 11: R3 -> R30
- J1_13 pad 14: R4 -> R29
- J1_13 pad 15: R4 -> R29
- J1_13 pad 18: R5 -> R28
- J1_13 pad 19: R5 -> R28
- J1_13 pad 2: R1 -> R32
- J1_13 pad 22: R6 -> R27
- J1_13 pad 23: R6 -> R27
- J1_13 pad 26: R7 -> R26
- J1_13 pad 27: R7 -> R26
- J1_13 pad 3: R1 -> R32
- J1_13 pad 30: R8 -> R25
- J1_13 pad 31: R8 -> R25
- J1_13 pad 34: R9 -> R24
- J1_13 pad 35: R9 -> R24
- J1_13 pad 38: R10 -> R23
- J1_13 pad 39: R10 -> R23
- J1_13 pad 42: R11 -> R22
- J1_13 pad 43: R11 -> R22
- J1_13 pad 46: R12 -> R21
- J1_13 pad 47: R12 -> R21
- J1_13 pad 50: R13 -> R20
- J1_13 pad 51: R13 -> R20
- J1_13 pad 54: R14 -> R19
- J1_13 pad 55: R14 -> R19
- J1_13 pad 58: R15 -> R18
- J1_13 pad 59: R15 -> R18
- J1_13 pad 6: R2 -> R31
- J1_13 pad 62: R16 -> R17
- J1_13 pad 63: R16 -> R17
- J1_13 pad 66: R17 -> R16
- J1_13 pad 67: R17 -> R16
- J1_13 pad 7: R2 -> R31
- J1_13 pad 70: R18 -> R15
- J1_13 pad 71: R18 -> R15
- J1_13 pad 74: R19 -> R14
- J1_13 pad 75: R19 -> R14
- J1_13 pad 78: R20 -> R13
- J1_13 pad 79: R20 -> R13
- J1_14 pad 10: R3 -> R30
- J1_14 pad 11: R3 -> R30
- J1_14 pad 14: R4 -> R29
- J1_14 pad 15: R4 -> R29
- J1_14 pad 18: R5 -> R28
- J1_14 pad 19: R5 -> R28
- J1_14 pad 2: R1 -> R32
- J1_14 pad 22: R6 -> R27
- J1_14 pad 23: R6 -> R27
- J1_14 pad 26: R7 -> R26
- J1_14 pad 27: R7 -> R26
- J1_14 pad 3: R1 -> R32
- J1_14 pad 30: R8 -> R25
- J1_14 pad 31: R8 -> R25
- J1_14 pad 34: R9 -> R24
- J1_14 pad 35: R9 -> R24
- J1_14 pad 38: R10 -> R23
- J1_14 pad 39: R10 -> R23
- J1_14 pad 42: R11 -> R22
- J1_14 pad 43: R11 -> R22
- J1_14 pad 46: R12 -> R21
- J1_14 pad 47: R12 -> R21
- J1_14 pad 50: R13 -> R20
- J1_14 pad 51: R13 -> R20
- J1_14 pad 54: R14 -> R19
- J1_14 pad 55: R14 -> R19
- J1_14 pad 58: R15 -> R18
- J1_14 pad 59: R15 -> R18
- J1_14 pad 6: R2 -> R31
- J1_14 pad 62: R16 -> R17
- J1_14 pad 63: R16 -> R17
- J1_14 pad 66: R17 -> R16
- J1_14 pad 67: R17 -> R16
- J1_14 pad 7: R2 -> R31
- J1_14 pad 70: R18 -> R15
- J1_14 pad 71: R18 -> R15
- J1_14 pad 74: R19 -> R14
- J1_14 pad 75: R19 -> R14
- J1_14 pad 78: R20 -> R13
- J1_14 pad 79: R20 -> R13
- J1_15 pad 10: R3 -> R30
- J1_15 pad 11: R3 -> R30
- J1_15 pad 14: R4 -> R29
- J1_15 pad 15: R4 -> R29
- J1_15 pad 18: R5 -> R28
- J1_15 pad 19: R5 -> R28
- J1_15 pad 2: R1 -> R32
- J1_15 pad 22: R6 -> R27
- J1_15 pad 23: R6 -> R27
- J1_15 pad 26: R7 -> R26
- J1_15 pad 27: R7 -> R26
- J1_15 pad 3: R1 -> R32
- J1_15 pad 30: R8 -> R25
- J1_15 pad 31: R8 -> R25
- J1_15 pad 34: R9 -> R24
- J1_15 pad 35: R9 -> R24
- J1_15 pad 38: R10 -> R23
- J1_15 pad 39: R10 -> R23
- J1_15 pad 42: R11 -> R22
- J1_15 pad 43: R11 -> R22
- J1_15 pad 46: R12 -> R21
- J1_15 pad 47: R12 -> R21
- J1_15 pad 50: R13 -> R20
- J1_15 pad 51: R13 -> R20
- J1_15 pad 54: R14 -> R19
- J1_15 pad 55: R14 -> R19
- J1_15 pad 58: R15 -> R18
- J1_15 pad 59: R15 -> R18
- J1_15 pad 6: R2 -> R31
- J1_15 pad 62: R16 -> R17
- J1_15 pad 63: R16 -> R17
- J1_15 pad 66: R17 -> R16
- J1_15 pad 67: R17 -> R16
- J1_15 pad 7: R2 -> R31
- J1_15 pad 70: R18 -> R15
- J1_15 pad 71: R18 -> R15
- J1_15 pad 74: R19 -> R14
- J1_15 pad 75: R19 -> R14
- J1_15 pad 78: R20 -> R13
- J1_15 pad 79: R20 -> R13
- J1_16 pad 10: R3 -> R30
- J1_16 pad 11: R3 -> R30
- J1_16 pad 14: R4 -> R29
- J1_16 pad 15: R4 -> R29
- J1_16 pad 18: R5 -> R28
- J1_16 pad 19: R5 -> R28
- J1_16 pad 2: R1 -> R32
- J1_16 pad 22: R6 -> R27
- J1_16 pad 23: R6 -> R27
- J1_16 pad 26: R7 -> R26
- J1_16 pad 27: R7 -> R26
- J1_16 pad 3: R1 -> R32
- J1_16 pad 30: R8 -> R25
- J1_16 pad 31: R8 -> R25
- J1_16 pad 34: R9 -> R24
- J1_16 pad 35: R9 -> R24
- J1_16 pad 38: R10 -> R23
- J1_16 pad 39: R10 -> R23
- J1_16 pad 42: R11 -> R22
- J1_16 pad 43: R11 -> R22
- J1_16 pad 46: R12 -> R21
- J1_16 pad 47: R12 -> R21
- J1_16 pad 50: R13 -> R20
- J1_16 pad 51: R13 -> R20
- J1_16 pad 54: R14 -> R19
- J1_16 pad 55: R14 -> R19
- J1_16 pad 58: R15 -> R18
- J1_16 pad 59: R15 -> R18
- J1_16 pad 6: R2 -> R31
- J1_16 pad 62: R16 -> R17
- J1_16 pad 63: R16 -> R17
- J1_16 pad 66: R17 -> R16
- J1_16 pad 67: R17 -> R16
- J1_16 pad 7: R2 -> R31
- J1_16 pad 70: R18 -> R15
- J1_16 pad 71: R18 -> R15
- J1_16 pad 74: R19 -> R14
- J1_16 pad 75: R19 -> R14
- J1_16 pad 78: R20 -> R13
- J1_16 pad 79: R20 -> R13
- J1_17 pad 10: R3 -> R30
- J1_17 pad 11: R3 -> R30
- J1_17 pad 14: R4 -> R29
- J1_17 pad 15: R4 -> R29
- J1_17 pad 18: R5 -> R28
- J1_17 pad 19: R5 -> R28
- J1_17 pad 2: R1 -> R32
- J1_17 pad 22: R6 -> R27
- J1_17 pad 23: R6 -> R27
- J1_17 pad 26: R7 -> R26
- J1_17 pad 27: R7 -> R26
- J1_17 pad 3: R1 -> R32
- J1_17 pad 30: R8 -> R25
- J1_17 pad 31: R8 -> R25
- J1_17 pad 34: R9 -> R24
- J1_17 pad 35: R9 -> R24
- J1_17 pad 38: R10 -> R23
- J1_17 pad 39: R10 -> R23
- J1_17 pad 42: R11 -> R22
- J1_17 pad 43: R11 -> R22
- J1_17 pad 46: R12 -> R21
- J1_17 pad 47: R12 -> R21
- J1_17 pad 50: R13 -> R20
- J1_17 pad 51: R13 -> R20
- J1_17 pad 54: R14 -> R19
- J1_17 pad 55: R14 -> R19
- J1_17 pad 58: R15 -> R18
- J1_17 pad 59: R15 -> R18
- J1_17 pad 6: R2 -> R31
- J1_17 pad 62: R16 -> R17
- J1_17 pad 63: R16 -> R17
- J1_17 pad 66: R17 -> R16
- J1_17 pad 67: R17 -> R16
- J1_17 pad 7: R2 -> R31
- J1_17 pad 70: R18 -> R15
- J1_17 pad 71: R18 -> R15
- J1_17 pad 74: R19 -> R14
- J1_17 pad 75: R19 -> R14
- J1_17 pad 78: R20 -> R13
- J1_17 pad 79: R20 -> R13
- J1_18 pad 10: R3 -> R30
- J1_18 pad 11: R3 -> R30
- J1_18 pad 14: R4 -> R29
- J1_18 pad 15: R4 -> R29
- J1_18 pad 18: R5 -> R28
- J1_18 pad 19: R5 -> R28
- J1_18 pad 2: R1 -> R32
- J1_18 pad 22: R6 -> R27
- J1_18 pad 23: R6 -> R27
- J1_18 pad 26: R7 -> R26
- J1_18 pad 27: R7 -> R26
- J1_18 pad 3: R1 -> R32
- J1_18 pad 30: R8 -> R25
- J1_18 pad 31: R8 -> R25
- J1_18 pad 34: R9 -> R24
- J1_18 pad 35: R9 -> R24
- J1_18 pad 38: R10 -> R23
- J1_18 pad 39: R10 -> R23
- J1_18 pad 42: R11 -> R22
- J1_18 pad 43: R11 -> R22
- J1_18 pad 46: R12 -> R21
- J1_18 pad 47: R12 -> R21
- J1_18 pad 50: R13 -> R20
- J1_18 pad 51: R13 -> R20
- J1_18 pad 54: R14 -> R19
- J1_18 pad 55: R14 -> R19
- J1_18 pad 58: R15 -> R18
- J1_18 pad 59: R15 -> R18
- J1_18 pad 6: R2 -> R31
- J1_18 pad 62: R16 -> R17
- J1_18 pad 63: R16 -> R17
- J1_18 pad 66: R17 -> R16
- J1_18 pad 67: R17 -> R16
- J1_18 pad 7: R2 -> R31
- J1_18 pad 70: R18 -> R15
- J1_18 pad 71: R18 -> R15
- J1_18 pad 74: R19 -> R14
- J1_18 pad 75: R19 -> R14
- J1_18 pad 78: R20 -> R13
- J1_18 pad 79: R20 -> R13
- J1_19 pad 10: R3 -> R30
- J1_19 pad 11: R3 -> R30
- J1_19 pad 14: R4 -> R29
- J1_19 pad 15: R4 -> R29
- J1_19 pad 18: R5 -> R28
- J1_19 pad 19: R5 -> R28
- J1_19 pad 2: R1 -> R32
- J1_19 pad 22: R6 -> R27
- J1_19 pad 23: R6 -> R27
- J1_19 pad 26: R7 -> R26
- J1_19 pad 27: R7 -> R26
- J1_19 pad 3: R1 -> R32
- J1_19 pad 30: R8 -> R25
- J1_19 pad 31: R8 -> R25
- J1_19 pad 34: R9 -> R24
- J1_19 pad 35: R9 -> R24
- J1_19 pad 38: R10 -> R23
- J1_19 pad 39: R10 -> R23
- J1_19 pad 42: R11 -> R22
- J1_19 pad 43: R11 -> R22
- J1_19 pad 46: R12 -> R21
- J1_19 pad 47: R12 -> R21
- J1_19 pad 50: R13 -> R20
- J1_19 pad 51: R13 -> R20
- J1_19 pad 54: R14 -> R19
- J1_19 pad 55: R14 -> R19
- J1_19 pad 58: R15 -> R18
- J1_19 pad 59: R15 -> R18
- J1_19 pad 6: R2 -> R31
- J1_19 pad 62: R16 -> R17
- J1_19 pad 63: R16 -> R17
- J1_19 pad 66: R17 -> R16
- J1_19 pad 67: R17 -> R16
- J1_19 pad 7: R2 -> R31
- J1_19 pad 70: R18 -> R15
- J1_19 pad 71: R18 -> R15
- J1_19 pad 74: R19 -> R14
- J1_19 pad 75: R19 -> R14
- J1_19 pad 78: R20 -> R13
- J1_19 pad 79: R20 -> R13
- J1_20 pad 10: R3 -> R30
- J1_20 pad 11: R3 -> R30
- J1_20 pad 14: R4 -> R29
- J1_20 pad 15: R4 -> R29
- J1_20 pad 18: R5 -> R28
- J1_20 pad 19: R5 -> R28
- J1_20 pad 2: R1 -> R32
- J1_20 pad 22: R6 -> R27
- J1_20 pad 23: R6 -> R27
- J1_20 pad 26: R7 -> R26
- J1_20 pad 27: R7 -> R26
- J1_20 pad 3: R1 -> R32
- J1_20 pad 30: R8 -> R25
- J1_20 pad 31: R8 -> R25
- J1_20 pad 34: R9 -> R24
- J1_20 pad 35: R9 -> R24
- J1_20 pad 38: R10 -> R23
- J1_20 pad 39: R10 -> R23
- J1_20 pad 42: R11 -> R22
- J1_20 pad 43: R11 -> R22
- J1_20 pad 46: R12 -> R21
- J1_20 pad 47: R12 -> R21
- J1_20 pad 50: R13 -> R20
- J1_20 pad 51: R13 -> R20
- J1_20 pad 54: R14 -> R19
- J1_20 pad 55: R14 -> R19
- J1_20 pad 58: R15 -> R18
- J1_20 pad 59: R15 -> R18
- J1_20 pad 6: R2 -> R31
- J1_20 pad 62: R16 -> R17
- J1_20 pad 63: R16 -> R17
- J1_20 pad 66: R17 -> R16
- J1_20 pad 67: R17 -> R16
- J1_20 pad 7: R2 -> R31
- J1_20 pad 70: R18 -> R15
- J1_20 pad 71: R18 -> R15
- J1_20 pad 74: R19 -> R14
- J1_20 pad 75: R19 -> R14
- J1_20 pad 78: R20 -> R13
- J1_20 pad 79: R20 -> R13
- J1_21 pad 10: R3 -> R30
- J1_21 pad 11: R3 -> R30
- J1_21 pad 14: R4 -> R29
- J1_21 pad 15: R4 -> R29
- J1_21 pad 18: R5 -> R28
- J1_21 pad 19: R5 -> R28
- J1_21 pad 2: R1 -> R32
- J1_21 pad 22: R6 -> R27
- J1_21 pad 23: R6 -> R27
- J1_21 pad 26: R7 -> R26
- J1_21 pad 27: R7 -> R26
- J1_21 pad 3: R1 -> R32
- J1_21 pad 30: R8 -> R25
- J1_21 pad 31: R8 -> R25
- J1_21 pad 34: R9 -> R24
- J1_21 pad 35: R9 -> R24
- J1_21 pad 38: R10 -> R23
- J1_21 pad 39: R10 -> R23
- J1_21 pad 42: R11 -> R22
- J1_21 pad 43: R11 -> R22
- J1_21 pad 46: R12 -> R21
- J1_21 pad 47: R12 -> R21
- J1_21 pad 50: R13 -> R20
- J1_21 pad 51: R13 -> R20
- J1_21 pad 54: R14 -> R19
- J1_21 pad 55: R14 -> R19
- J1_21 pad 58: R15 -> R18
- J1_21 pad 59: R15 -> R18
- J1_21 pad 6: R2 -> R31
- J1_21 pad 62: R16 -> R17
- J1_21 pad 63: R16 -> R17
- J1_21 pad 66: R17 -> R16
- J1_21 pad 67: R17 -> R16
- J1_21 pad 7: R2 -> R31
- J1_21 pad 70: R18 -> R15
- J1_21 pad 71: R18 -> R15
- J1_21 pad 74: R19 -> R14
- J1_21 pad 75: R19 -> R14
- J1_21 pad 78: R20 -> R13
- J1_21 pad 79: R20 -> R13
- J1_22 pad 10: R3 -> R30
- J1_22 pad 11: R3 -> R30
- J1_22 pad 14: R4 -> R29
- J1_22 pad 15: R4 -> R29
- J1_22 pad 18: R5 -> R28
- J1_22 pad 19: R5 -> R28
- J1_22 pad 2: R1 -> R32
- J1_22 pad 22: R6 -> R27
- J1_22 pad 23: R6 -> R27
- J1_22 pad 26: R7 -> R26
- J1_22 pad 27: R7 -> R26
- J1_22 pad 3: R1 -> R32
- J1_22 pad 30: R8 -> R25
- J1_22 pad 31: R8 -> R25
- J1_22 pad 34: R9 -> R24
- J1_22 pad 35: R9 -> R24
- J1_22 pad 38: R10 -> R23
- J1_22 pad 39: R10 -> R23
- J1_22 pad 42: R11 -> R22
- J1_22 pad 43: R11 -> R22
- J1_22 pad 46: R12 -> R21
- J1_22 pad 47: R12 -> R21
- J1_22 pad 50: R13 -> R20
- J1_22 pad 51: R13 -> R20
- J1_22 pad 54: R14 -> R19
- J1_22 pad 55: R14 -> R19
- J1_22 pad 58: R15 -> R18
- J1_22 pad 59: R15 -> R18
- J1_22 pad 6: R2 -> R31
- J1_22 pad 62: R16 -> R17
- J1_22 pad 63: R16 -> R17
- J1_22 pad 66: R17 -> R16
- J1_22 pad 67: R17 -> R16
- J1_22 pad 7: R2 -> R31
- J1_22 pad 70: R18 -> R15
- J1_22 pad 71: R18 -> R15
- J1_22 pad 74: R19 -> R14
- J1_22 pad 75: R19 -> R14
- J1_22 pad 78: R20 -> R13
- J1_22 pad 79: R20 -> R13
- J1_23 pad 10: R3 -> R30
- J1_23 pad 11: R3 -> R30
- J1_23 pad 14: R4 -> R29
- J1_23 pad 15: R4 -> R29
- J1_23 pad 18: R5 -> R28
- J1_23 pad 19: R5 -> R28
- J1_23 pad 2: R1 -> R32
- J1_23 pad 22: R6 -> R27
- J1_23 pad 23: R6 -> R27
- J1_23 pad 26: R7 -> R26
- J1_23 pad 27: R7 -> R26
- J1_23 pad 3: R1 -> R32
- J1_23 pad 30: R8 -> R25
- J1_23 pad 31: R8 -> R25
- J1_23 pad 34: R9 -> R24
- J1_23 pad 35: R9 -> R24
- J1_23 pad 38: R10 -> R23
- J1_23 pad 39: R10 -> R23
- J1_23 pad 42: R11 -> R22
- J1_23 pad 43: R11 -> R22
- J1_23 pad 46: R12 -> R21
- J1_23 pad 47: R12 -> R21
- J1_23 pad 50: R13 -> R20
- J1_23 pad 51: R13 -> R20
- J1_23 pad 54: R14 -> R19
- J1_23 pad 55: R14 -> R19
- J1_23 pad 58: R15 -> R18
- J1_23 pad 59: R15 -> R18
- J1_23 pad 6: R2 -> R31
- J1_23 pad 62: R16 -> R17
- J1_23 pad 63: R16 -> R17
- J1_23 pad 66: R17 -> R16
- J1_23 pad 67: R17 -> R16
- J1_23 pad 7: R2 -> R31
- J1_23 pad 70: R18 -> R15
- J1_23 pad 71: R18 -> R15
- J1_23 pad 74: R19 -> R14
- J1_23 pad 75: R19 -> R14
- J1_23 pad 78: R20 -> R13
- J1_23 pad 79: R20 -> R13
- J1_24 pad 10: R3 -> R30
- J1_24 pad 11: R3 -> R30
- J1_24 pad 14: R4 -> R29
- J1_24 pad 15: R4 -> R29
- J1_24 pad 18: R5 -> R28
- J1_24 pad 19: R5 -> R28
- J1_24 pad 2: R1 -> R32
- J1_24 pad 22: R6 -> R27
- J1_24 pad 23: R6 -> R27
- J1_24 pad 26: R7 -> R26
- J1_24 pad 27: R7 -> R26
- J1_24 pad 3: R1 -> R32
- J1_24 pad 30: R8 -> R25
- J1_24 pad 31: R8 -> R25
- J1_24 pad 34: R9 -> R24
- J1_24 pad 35: R9 -> R24
- J1_24 pad 38: R10 -> R23
- J1_24 pad 39: R10 -> R23
- J1_24 pad 42: R11 -> R22
- J1_24 pad 43: R11 -> R22
- J1_24 pad 46: R12 -> R21
- J1_24 pad 47: R12 -> R21
- J1_24 pad 50: R13 -> R20
- J1_24 pad 51: R13 -> R20
- J1_24 pad 54: R14 -> R19
- J1_24 pad 55: R14 -> R19
- J1_24 pad 58: R15 -> R18
- J1_24 pad 59: R15 -> R18
- J1_24 pad 6: R2 -> R31
- J1_24 pad 62: R16 -> R17
- J1_24 pad 63: R16 -> R17
- J1_24 pad 66: R17 -> R16
- J1_24 pad 67: R17 -> R16
- J1_24 pad 7: R2 -> R31
- J1_24 pad 70: R18 -> R15
- J1_24 pad 71: R18 -> R15
- J1_24 pad 74: R19 -> R14
- J1_24 pad 75: R19 -> R14
- J1_24 pad 78: R20 -> R13
- J1_24 pad 79: R20 -> R13
- J1_25 pad 10: R3 -> R30
- J1_25 pad 11: R3 -> R30
- J1_25 pad 14: R4 -> R29
- J1_25 pad 15: R4 -> R29
- J1_25 pad 18: R5 -> R28
- J1_25 pad 19: R5 -> R28
- J1_25 pad 2: R1 -> R32
- J1_25 pad 22: R6 -> R27
- J1_25 pad 23: R6 -> R27
- J1_25 pad 26: R7 -> R26
- J1_25 pad 27: R7 -> R26
- J1_25 pad 3: R1 -> R32
- J1_25 pad 30: R8 -> R25
- J1_25 pad 31: R8 -> R25
- J1_25 pad 34: R9 -> R24
- J1_25 pad 35: R9 -> R24
- J1_25 pad 38: R10 -> R23
- J1_25 pad 39: R10 -> R23
- J1_25 pad 42: R11 -> R22
- J1_25 pad 43: R11 -> R22
- J1_25 pad 46: R12 -> R21
- J1_25 pad 47: R12 -> R21
- J1_25 pad 50: R13 -> R20
- J1_25 pad 51: R13 -> R20
- J1_25 pad 54: R14 -> R19
- J1_25 pad 55: R14 -> R19
- J1_25 pad 58: R15 -> R18
- J1_25 pad 59: R15 -> R18
- J1_25 pad 6: R2 -> R31
- J1_25 pad 62: R16 -> R17
- J1_25 pad 63: R16 -> R17
- J1_25 pad 66: R17 -> R16
- J1_25 pad 67: R17 -> R16
- J1_25 pad 7: R2 -> R31
- J1_25 pad 70: R18 -> R15
- J1_25 pad 71: R18 -> R15
- J1_25 pad 74: R19 -> R14
- J1_25 pad 75: R19 -> R14
- J1_25 pad 78: R20 -> R13
- J1_25 pad 79: R20 -> R13
- J1_26 pad 10: R3 -> R30
- J1_26 pad 11: R3 -> R30
- J1_26 pad 14: R4 -> R29
- J1_26 pad 15: R4 -> R29
- J1_26 pad 18: R5 -> R28
- J1_26 pad 19: R5 -> R28
- J1_26 pad 2: R1 -> R32
- J1_26 pad 22: R6 -> R27
- J1_26 pad 23: R6 -> R27
- J1_26 pad 26: R7 -> R26
- J1_26 pad 27: R7 -> R26
- J1_26 pad 3: R1 -> R32
- J1_26 pad 30: R8 -> R25
- J1_26 pad 31: R8 -> R25
- J1_26 pad 34: R9 -> R24
- J1_26 pad 35: R9 -> R24
- J1_26 pad 38: R10 -> R23
- J1_26 pad 39: R10 -> R23
- J1_26 pad 42: R11 -> R22
- J1_26 pad 43: R11 -> R22
- J1_26 pad 46: R12 -> R21
- J1_26 pad 47: R12 -> R21
- J1_26 pad 50: R13 -> R20
- J1_26 pad 51: R13 -> R20
- J1_26 pad 54: R14 -> R19
- J1_26 pad 55: R14 -> R19
- J1_26 pad 58: R15 -> R18
- J1_26 pad 59: R15 -> R18
- J1_26 pad 6: R2 -> R31
- J1_26 pad 62: R16 -> R17
- J1_26 pad 63: R16 -> R17
- J1_26 pad 66: R17 -> R16
- J1_26 pad 67: R17 -> R16
- J1_26 pad 7: R2 -> R31
- J1_26 pad 70: R18 -> R15
- J1_26 pad 71: R18 -> R15
- J1_26 pad 74: R19 -> R14
- J1_26 pad 75: R19 -> R14
- J1_26 pad 78: R20 -> R13
- J1_26 pad 79: R20 -> R13
- J1_27 pad 10: R3 -> R30
- J1_27 pad 11: R3 -> R30
- J1_27 pad 14: R4 -> R29
- J1_27 pad 15: R4 -> R29
- J1_27 pad 18: R5 -> R28
- J1_27 pad 19: R5 -> R28
- J1_27 pad 2: R1 -> R32
- J1_27 pad 22: R6 -> R27
- J1_27 pad 23: R6 -> R27
- J1_27 pad 26: R7 -> R26
- J1_27 pad 27: R7 -> R26
- J1_27 pad 3: R1 -> R32
- J1_27 pad 30: R8 -> R25
- J1_27 pad 31: R8 -> R25
- J1_27 pad 34: R9 -> R24
- J1_27 pad 35: R9 -> R24
- J1_27 pad 38: R10 -> R23
- J1_27 pad 39: R10 -> R23
- J1_27 pad 42: R11 -> R22
- J1_27 pad 43: R11 -> R22
- J1_27 pad 46: R12 -> R21
- J1_27 pad 47: R12 -> R21
- J1_27 pad 50: R13 -> R20
- J1_27 pad 51: R13 -> R20
- J1_27 pad 54: R14 -> R19
- J1_27 pad 55: R14 -> R19
- J1_27 pad 58: R15 -> R18
- J1_27 pad 59: R15 -> R18
- J1_27 pad 6: R2 -> R31
- J1_27 pad 62: R16 -> R17
- J1_27 pad 63: R16 -> R17
- J1_27 pad 66: R17 -> R16
- J1_27 pad 67: R17 -> R16
- J1_27 pad 7: R2 -> R31
- J1_27 pad 70: R18 -> R15
- J1_27 pad 71: R18 -> R15
- J1_27 pad 74: R19 -> R14
- J1_27 pad 75: R19 -> R14
- J1_27 pad 78: R20 -> R13
- J1_27 pad 79: R20 -> R13
- J1_28 pad 10: R3 -> R30
- J1_28 pad 11: R3 -> R30
- J1_28 pad 14: R4 -> R29
- J1_28 pad 15: R4 -> R29
- J1_28 pad 18: R5 -> R28
- J1_28 pad 19: R5 -> R28
- J1_28 pad 2: R1 -> R32
- J1_28 pad 22: R6 -> R27
- J1_28 pad 23: R6 -> R27
- J1_28 pad 26: R7 -> R26
- J1_28 pad 27: R7 -> R26
- J1_28 pad 3: R1 -> R32
- J1_28 pad 30: R8 -> R25
- J1_28 pad 31: R8 -> R25
- J1_28 pad 34: R9 -> R24
- J1_28 pad 35: R9 -> R24
- J1_28 pad 38: R10 -> R23
- J1_28 pad 39: R10 -> R23
- J1_28 pad 42: R11 -> R22
- J1_28 pad 43: R11 -> R22
- J1_28 pad 46: R12 -> R21
- J1_28 pad 47: R12 -> R21
- J1_28 pad 50: R13 -> R20
- J1_28 pad 51: R13 -> R20
- J1_28 pad 54: R14 -> R19
- J1_28 pad 55: R14 -> R19
- J1_28 pad 58: R15 -> R18
- J1_28 pad 59: R15 -> R18
- J1_28 pad 6: R2 -> R31
- J1_28 pad 62: R16 -> R17
- J1_28 pad 63: R16 -> R17
- J1_28 pad 66: R17 -> R16
- J1_28 pad 67: R17 -> R16
- J1_28 pad 7: R2 -> R31
- J1_28 pad 70: R18 -> R15
- J1_28 pad 71: R18 -> R15
- J1_28 pad 74: R19 -> R14
- J1_28 pad 75: R19 -> R14
- J1_28 pad 78: R20 -> R13
- J1_28 pad 79: R20 -> R13
- J1_29 pad 10: R3 -> R30
- J1_29 pad 11: R3 -> R30
- J1_29 pad 14: R4 -> R29
- J1_29 pad 15: R4 -> R29
- J1_29 pad 18: R5 -> R28
- J1_29 pad 19: R5 -> R28
- J1_29 pad 2: R1 -> R32
- J1_29 pad 22: R6 -> R27
- J1_29 pad 23: R6 -> R27
- J1_29 pad 26: R7 -> R26
- J1_29 pad 27: R7 -> R26
- J1_29 pad 3: R1 -> R32
- J1_29 pad 30: R8 -> R25
- J1_29 pad 31: R8 -> R25
- J1_29 pad 34: R9 -> R24
- J1_29 pad 35: R9 -> R24
- J1_29 pad 38: R10 -> R23
- J1_29 pad 39: R10 -> R23
- J1_29 pad 42: R11 -> R22
- J1_29 pad 43: R11 -> R22
- J1_29 pad 46: R12 -> R21
- J1_29 pad 47: R12 -> R21
- J1_29 pad 50: R13 -> R20
- J1_29 pad 51: R13 -> R20
- J1_29 pad 54: R14 -> R19
- J1_29 pad 55: R14 -> R19
- J1_29 pad 58: R15 -> R18
- J1_29 pad 59: R15 -> R18
- J1_29 pad 6: R2 -> R31
- J1_29 pad 62: R16 -> R17
- J1_29 pad 63: R16 -> R17
- J1_29 pad 66: R17 -> R16
- J1_29 pad 67: R17 -> R16
- J1_29 pad 7: R2 -> R31
- J1_29 pad 70: R18 -> R15
- J1_29 pad 71: R18 -> R15
- J1_29 pad 74: R19 -> R14
- J1_29 pad 75: R19 -> R14
- J1_29 pad 78: R20 -> R13
- J1_29 pad 79: R20 -> R13
- J1_30 pad 10: R3 -> R30
- J1_30 pad 11: R3 -> R30
- J1_30 pad 14: R4 -> R29
- J1_30 pad 15: R4 -> R29
- J1_30 pad 18: R5 -> R28
- J1_30 pad 19: R5 -> R28
- J1_30 pad 2: R1 -> R32
- J1_30 pad 22: R6 -> R27
- J1_30 pad 23: R6 -> R27
- J1_30 pad 26: R7 -> R26
- J1_30 pad 27: R7 -> R26
- J1_30 pad 3: R1 -> R32
- J1_30 pad 30: R8 -> R25
- J1_30 pad 31: R8 -> R25
- J1_30 pad 34: R9 -> R24
- J1_30 pad 35: R9 -> R24
- J1_30 pad 38: R10 -> R23
- J1_30 pad 39: R10 -> R23
- J1_30 pad 42: R11 -> R22
- J1_30 pad 43: R11 -> R22
- J1_30 pad 46: R12 -> R21
- J1_30 pad 47: R12 -> R21
- J1_30 pad 50: R13 -> R20
- J1_30 pad 51: R13 -> R20
- J1_30 pad 54: R14 -> R19
- J1_30 pad 55: R14 -> R19
- J1_30 pad 58: R15 -> R18
- J1_30 pad 59: R15 -> R18
- J1_30 pad 6: R2 -> R31
- J1_30 pad 62: R16 -> R17
- J1_30 pad 63: R16 -> R17
- J1_30 pad 66: R17 -> R16
- J1_30 pad 67: R17 -> R16
- J1_30 pad 7: R2 -> R31
- J1_30 pad 70: R18 -> R15
- J1_30 pad 71: R18 -> R15
- J1_30 pad 74: R19 -> R14
- J1_30 pad 75: R19 -> R14
- J1_30 pad 78: R20 -> R13
- J1_30 pad 79: R20 -> R13
- J1_31 pad 10: R3 -> R30
- J1_31 pad 11: R3 -> R30
- J1_31 pad 14: R4 -> R29
- J1_31 pad 15: R4 -> R29
- J1_31 pad 18: R5 -> R28
- J1_31 pad 19: R5 -> R28
- J1_31 pad 2: R1 -> R32
- J1_31 pad 22: R6 -> R27
- J1_31 pad 23: R6 -> R27
- J1_31 pad 26: R7 -> R26
- J1_31 pad 27: R7 -> R26
- J1_31 pad 3: R1 -> R32
- J1_31 pad 30: R8 -> R25
- J1_31 pad 31: R8 -> R25
- J1_31 pad 34: R9 -> R24
- J1_31 pad 35: R9 -> R24
- J1_31 pad 38: R10 -> R23
- J1_31 pad 39: R10 -> R23
- J1_31 pad 42: R11 -> R22
- J1_31 pad 43: R11 -> R22
- J1_31 pad 46: R12 -> R21
- J1_31 pad 47: R12 -> R21
- J1_31 pad 50: R13 -> R20
- J1_31 pad 51: R13 -> R20
- J1_31 pad 54: R14 -> R19
- J1_31 pad 55: R14 -> R19
- J1_31 pad 58: R15 -> R18
- J1_31 pad 59: R15 -> R18
- J1_31 pad 6: R2 -> R31
- J1_31 pad 62: R16 -> R17
- J1_31 pad 63: R16 -> R17
- J1_31 pad 66: R17 -> R16
- J1_31 pad 67: R17 -> R16
- J1_31 pad 7: R2 -> R31
- J1_31 pad 70: R18 -> R15
- J1_31 pad 71: R18 -> R15
- J1_31 pad 74: R19 -> R14
- J1_31 pad 75: R19 -> R14
- J1_31 pad 78: R20 -> R13
- J1_31 pad 79: R20 -> R13
- J1_32 pad 10: R3 -> R30
- J1_32 pad 11: R3 -> R30
- J1_32 pad 14: R4 -> R29
- J1_32 pad 15: R4 -> R29
- J1_32 pad 18: R5 -> R28
- J1_32 pad 19: R5 -> R28
- J1_32 pad 2: R1 -> R32
- J1_32 pad 22: R6 -> R27
- J1_32 pad 23: R6 -> R27
- J1_32 pad 26: R7 -> R26
- J1_32 pad 27: R7 -> R26
- J1_32 pad 3: R1 -> R32
- J1_32 pad 30: R8 -> R25
- J1_32 pad 31: R8 -> R25
- J1_32 pad 34: R9 -> R24
- J1_32 pad 35: R9 -> R24
- J1_32 pad 38: R10 -> R23
- J1_32 pad 39: R10 -> R23
- J1_32 pad 42: R11 -> R22
- J1_32 pad 43: R11 -> R22
- J1_32 pad 46: R12 -> R21
- J1_32 pad 47: R12 -> R21
- J1_32 pad 50: R13 -> R20
- J1_32 pad 51: R13 -> R20
- J1_32 pad 54: R14 -> R19
- J1_32 pad 55: R14 -> R19
- J1_32 pad 58: R15 -> R18
- J1_32 pad 59: R15 -> R18
- J1_32 pad 6: R2 -> R31
- J1_32 pad 62: R16 -> R17
- J1_32 pad 63: R16 -> R17
- J1_32 pad 66: R17 -> R16
- J1_32 pad 67: R17 -> R16
- J1_32 pad 7: R2 -> R31
- J1_32 pad 70: R18 -> R15
- J1_32 pad 71: R18 -> R15
- J1_32 pad 74: R19 -> R14
- J1_32 pad 75: R19 -> R14
- J1_32 pad 78: R20 -> R13
- J1_32 pad 79: R20 -> R13
- J2_01 pad 10: R23 -> R10
- J2_01 pad 11: R23 -> R10
- J2_01 pad 14: R24 -> R9
- J2_01 pad 15: R24 -> R9
- J2_01 pad 18: R25 -> R8
- J2_01 pad 19: R25 -> R8
- J2_01 pad 2: R21 -> R12
- J2_01 pad 22: R26 -> R7
- J2_01 pad 23: R26 -> R7
- J2_01 pad 26: R27 -> R6
- J2_01 pad 27: R27 -> R6
- J2_01 pad 3: R21 -> R12
- J2_01 pad 30: R28 -> R5
- J2_01 pad 31: R28 -> R5
- J2_01 pad 34: R29 -> R4
- J2_01 pad 35: R29 -> R4
- J2_01 pad 38: R30 -> R3
- J2_01 pad 39: R30 -> R3
- J2_01 pad 42: R31 -> R2
- J2_01 pad 43: R31 -> R2
- J2_01 pad 46: R32 -> R1
- J2_01 pad 47: R32 -> R1
- J2_01 pad 6: R22 -> R11
- J2_01 pad 7: R22 -> R11
- J2_02 pad 10: R23 -> R10
- J2_02 pad 11: R23 -> R10
- J2_02 pad 14: R24 -> R9
- J2_02 pad 15: R24 -> R9
- J2_02 pad 18: R25 -> R8
- J2_02 pad 19: R25 -> R8
- J2_02 pad 2: R21 -> R12
- J2_02 pad 22: R26 -> R7
- J2_02 pad 23: R26 -> R7
- J2_02 pad 26: R27 -> R6
- J2_02 pad 27: R27 -> R6
- J2_02 pad 3: R21 -> R12
- J2_02 pad 30: R28 -> R5
- J2_02 pad 31: R28 -> R5
- J2_02 pad 34: R29 -> R4
- J2_02 pad 35: R29 -> R4
- J2_02 pad 38: R30 -> R3
- J2_02 pad 39: R30 -> R3
- J2_02 pad 42: R31 -> R2
- J2_02 pad 43: R31 -> R2
- J2_02 pad 46: R32 -> R1
- J2_02 pad 47: R32 -> R1
- J2_02 pad 6: R22 -> R11
- J2_02 pad 7: R22 -> R11
- J2_03 pad 10: R23 -> R10
- J2_03 pad 11: R23 -> R10
- J2_03 pad 14: R24 -> R9
- J2_03 pad 15: R24 -> R9
- J2_03 pad 18: R25 -> R8
- J2_03 pad 19: R25 -> R8
- J2_03 pad 2: R21 -> R12
- J2_03 pad 22: R26 -> R7
- J2_03 pad 23: R26 -> R7
- J2_03 pad 26: R27 -> R6
- J2_03 pad 27: R27 -> R6
- J2_03 pad 3: R21 -> R12
- J2_03 pad 30: R28 -> R5
- J2_03 pad 31: R28 -> R5
- J2_03 pad 34: R29 -> R4
- J2_03 pad 35: R29 -> R4
- J2_03 pad 38: R30 -> R3
- J2_03 pad 39: R30 -> R3
- J2_03 pad 42: R31 -> R2
- J2_03 pad 43: R31 -> R2
- J2_03 pad 46: R32 -> R1
- J2_03 pad 47: R32 -> R1
- J2_03 pad 6: R22 -> R11
- J2_03 pad 7: R22 -> R11
- J2_04 pad 10: R23 -> R10
- J2_04 pad 11: R23 -> R10
- J2_04 pad 14: R24 -> R9
- J2_04 pad 15: R24 -> R9
- J2_04 pad 18: R25 -> R8
- J2_04 pad 19: R25 -> R8
- J2_04 pad 2: R21 -> R12
- J2_04 pad 22: R26 -> R7
- J2_04 pad 23: R26 -> R7
- J2_04 pad 26: R27 -> R6
- J2_04 pad 27: R27 -> R6
- J2_04 pad 3: R21 -> R12
- J2_04 pad 30: R28 -> R5
- J2_04 pad 31: R28 -> R5
- J2_04 pad 34: R29 -> R4
- J2_04 pad 35: R29 -> R4
- J2_04 pad 38: R30 -> R3
- J2_04 pad 39: R30 -> R3
- J2_04 pad 42: R31 -> R2
- J2_04 pad 43: R31 -> R2
- J2_04 pad 46: R32 -> R1
- J2_04 pad 47: R32 -> R1
- J2_04 pad 6: R22 -> R11
- J2_04 pad 7: R22 -> R11
- J2_05 pad 10: R23 -> R10
- J2_05 pad 11: R23 -> R10
- J2_05 pad 14: R24 -> R9
- J2_05 pad 15: R24 -> R9
- J2_05 pad 18: R25 -> R8
- J2_05 pad 19: R25 -> R8
- J2_05 pad 2: R21 -> R12
- J2_05 pad 22: R26 -> R7
- J2_05 pad 23: R26 -> R7
- J2_05 pad 26: R27 -> R6
- J2_05 pad 27: R27 -> R6
- J2_05 pad 3: R21 -> R12
- J2_05 pad 30: R28 -> R5
- J2_05 pad 31: R28 -> R5
- J2_05 pad 34: R29 -> R4
- J2_05 pad 35: R29 -> R4
- J2_05 pad 38: R30 -> R3
- J2_05 pad 39: R30 -> R3
- J2_05 pad 42: R31 -> R2
- J2_05 pad 43: R31 -> R2
- J2_05 pad 46: R32 -> R1
- J2_05 pad 47: R32 -> R1
- J2_05 pad 6: R22 -> R11
- J2_05 pad 7: R22 -> R11
- J2_06 pad 10: R23 -> R10
- J2_06 pad 11: R23 -> R10
- J2_06 pad 14: R24 -> R9
- J2_06 pad 15: R24 -> R9
- J2_06 pad 18: R25 -> R8
- J2_06 pad 19: R25 -> R8
- J2_06 pad 2: R21 -> R12
- J2_06 pad 22: R26 -> R7
- J2_06 pad 23: R26 -> R7
- J2_06 pad 26: R27 -> R6
- J2_06 pad 27: R27 -> R6
- J2_06 pad 3: R21 -> R12
- J2_06 pad 30: R28 -> R5
- J2_06 pad 31: R28 -> R5
- J2_06 pad 34: R29 -> R4
- J2_06 pad 35: R29 -> R4
- J2_06 pad 38: R30 -> R3
- J2_06 pad 39: R30 -> R3
- J2_06 pad 42: R31 -> R2
- J2_06 pad 43: R31 -> R2
- J2_06 pad 46: R32 -> R1
- J2_06 pad 47: R32 -> R1
- J2_06 pad 6: R22 -> R11
- J2_06 pad 7: R22 -> R11
- J2_07 pad 10: R23 -> R10
- J2_07 pad 11: R23 -> R10
- J2_07 pad 14: R24 -> R9
- J2_07 pad 15: R24 -> R9
- J2_07 pad 18: R25 -> R8
- J2_07 pad 19: R25 -> R8
- J2_07 pad 2: R21 -> R12
- J2_07 pad 22: R26 -> R7
- J2_07 pad 23: R26 -> R7
- J2_07 pad 26: R27 -> R6
- J2_07 pad 27: R27 -> R6
- J2_07 pad 3: R21 -> R12
- J2_07 pad 30: R28 -> R5
- J2_07 pad 31: R28 -> R5
- J2_07 pad 34: R29 -> R4
- J2_07 pad 35: R29 -> R4
- J2_07 pad 38: R30 -> R3
- J2_07 pad 39: R30 -> R3
- J2_07 pad 42: R31 -> R2
- J2_07 pad 43: R31 -> R2
- J2_07 pad 46: R32 -> R1
- J2_07 pad 47: R32 -> R1
- J2_07 pad 6: R22 -> R11
- J2_07 pad 7: R22 -> R11
- J2_08 pad 10: R23 -> R10
- J2_08 pad 11: R23 -> R10
- J2_08 pad 14: R24 -> R9
- J2_08 pad 15: R24 -> R9
- J2_08 pad 18: R25 -> R8
- J2_08 pad 19: R25 -> R8
- J2_08 pad 2: R21 -> R12
- J2_08 pad 22: R26 -> R7
- J2_08 pad 23: R26 -> R7
- J2_08 pad 26: R27 -> R6
- J2_08 pad 27: R27 -> R6
- J2_08 pad 3: R21 -> R12
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Routing:
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Other:
- outline, holes or cut-outs redrawn
- board text added: "servernoj/cheroma @ Github March 2026"
- board text removed: "@servernoj 03/26"
