File: CAD/KiCAD/digitizer/digitizer.kicad_pcb (KiCad board)
At the start: 2 copper layers, 254 x 254 mm, 80 parts, among them J1 Conn_01x06, J1_01 Conn_02x40_Odd_Even, J1_02 Conn_02x40_Odd_Even, J1_03 Conn_02x40_Odd_Even, J1_04 Conn_02x40_Odd_Even, J1_05 Conn_02x40_Odd_Even, J1_06 Conn_02x40_Odd_Even, J1_07 Conn_02x40_Odd_Even, J1_08 Conn_02x40_Odd_Even, J1_09 Conn_02x40_Odd_Even, J1_10 Conn_02x40_Odd_Even, J1_11 Conn_02x40_Odd_Even, J1_12 Conn_02x40_Odd_Even, J1_13 Conn_02x40_Odd_Even, J1_14 Conn_02x40_Odd_Even, J1_15 Conn_02x40_Odd_Even, J1_16 Conn_02x40_Odd_Even, J1_17 Conn_02x40_Odd_Even, J1_18 Conn_02x40_Odd_Even, J1_19 Conn_02x40_Odd_Even, J1_20 Conn_02x40_Odd_Even, J1_21 Conn_02x40_Odd_Even, J1_22 Conn_02x40_Odd_Even, J1_23 Conn_02x40_Odd_Even, J1_24 Conn_02x40_Odd_Even, J1_25 Conn_02x40_Odd_Even, J1_26 Conn_02x40_Odd_Even, J1_27 Conn_02x40_Odd_Even, J1_28 Conn_02x40_Odd_Even, J1_29 Conn_02x40_Odd_Even, J1_30 Conn_02x40_Odd_Even, J1_31 Conn_02x40_Odd_Even, J1_32 Conn_02x40_Odd_Even, J2 Conn_01x06, J2_01 Conn_02x24_Odd_Even, J2_02 Conn_02x24_Odd_Even, J2_03 Conn_02x24_Odd_Even, J2_04 Conn_02x24_Odd_Even, J2_05 Conn_02x24_Odd_Even, J2_06 Conn_02x24_Odd_Even, J2_07 Conn_02x24_Odd_Even, J2_08 Conn_02x24_Odd_Even, J2_09 Conn_02x24_Odd_Even, J2_10 Conn_02x24_Odd_Even, J2_11 Conn_02x24_Odd_Even, J2_12 Conn_02x24_Odd_Even, J2_13 Conn_02x24_Odd_Even, J2_14 Conn_02x24_Odd_Even, J2_15 Conn_02x24_Odd_Even, J2_16 Conn_02x24_Odd_Even, J2_17 Conn_02x24_Odd_Even, J2_18 Conn_02x24_Odd_Even, J2_19 Conn_02x24_Odd_Even, J2_20 Conn_02x24_Odd_Even, J2_21 Conn_02x24_Odd_Even, J2_22 Conn_02x24_Odd_Even, J2_23 Conn_02x24_Odd_Even, J2_24 Conn_02x24_Odd_Even, J2_25 Conn_02x24_Odd_Even, J2_26 Conn_02x24_Odd_Even, J2_27 Conn_02x24_Odd_Even, J2_28 Conn_02x24_Odd_Even, J2_29 Conn_02x24_Odd_Even, J2_30 Conn_02x24_Odd_Even, J2_31 Conn_02x24_Odd_Even, J2_32 Conn_02x24_Odd_Even, P1_1 Conn_01x06, P1_2 Conn_01x06, P1_3 Conn_01x06, P1_4 Conn_01x06, P3_1 Conn_01x10, P3_2 Conn_01x10, P3_3 Conn_01x10, P3_4 Conn_01x10, P4_1 Conn_01x10, P4_2 Conn_01x10, P4_3 Conn_01x10, P4_4 Conn_01x10

Commit message: cad: add pull-up resistors to interrupt lines
Parts:
- added R3: 10k, Resistor_THT:R_Axial_DIN0207_L6.3mm_D2.5mm_P15.24mm_Horizontal, F.Cu at (71.1, 182.6)
- added R4: 10k, Resistor_THT:R_Axial_DIN0207_L6.3mm_D2.5mm_P15.24mm_Horizontal, F.Cu at (71.1, 188.2)
- moved R1 8.89 mm to (71.1, 171.4)
- moved R2 8.33 mm to (71.1, 177.0)
Routing:
- net INTA: track 481.5 -> 524.8 mm
- net INTB: track 486.4 -> 520.5 mm
- net VCC: track 532.2 -> 546.9 mm
- net SDA: track 536.4 -> 533.6 mm

Commit message: digitizer integration draft take 1
Other:
- board text added: "v1.1"
- board text removed: "v1.0"
Changed lines of the file:
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@@
 		)
 	)
-	(gr_text "v1.0"
+	(gr_text "v1.1"
 		(at 71.628 51.308 0)
 		(layer "F.SilkS")
