File: CAD/KiCAD/digitizer/header_40x2.kicad_sch (KiCad schematic)
At the start: 1 part, among them J1 Conn_02x40_Odd_Even

Commit message: add MCP23017 for rows (no routing)
Parts:
- renumbered J1 to J7a
Changed lines of the file:
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@@
 		(on_board yes)
 		(dnp no)
-		(property "Reference" "J1"
+		(property "Reference" "J7a"
 			(at 76.2 40.64 0)
 			(effects
@@
 			(project "digitizer"
 				(path "/7204cdda-0a14-40c0-9dc8-8318dd514140/3d809a25-cc61-4069-acab-552aa888d46b/0a77984b-0e61-43a3-838f-8583936efe88"
-					(reference "J42")
+					(reference "J24a")
 					(unit 1)
 				)
 				(path "/7204cdda-0a14-40c0-9dc8-8318dd514140/3d809a25-cc61-4069-acab-552aa888d46b/316b265e-96e5-4e12-ba62-f527eb037ccf"
-					(reference "J43")
+					(reference "J21a")
 					(unit 1)
 				)
 				(path "/7204cdda-0a14-40c0-9dc8-8318dd514140/3d809a25-cc61-4069-acab-552aa888d46b/a5941889-9e91-48ac-996e-3109bbfd970a"
-					(reference "J44")
+					(reference "J22a")
 					(unit 1)
 				)
 				(path "/7204cdda-0a14-40c0-9dc8-8318dd514140/3d809a25-cc61-4069-acab-552aa888d46b/a6f8974c-4bb2-46a6-a2f5-229d9d791f49"
-					(reference "J41")
+					(reference "J23a")
 					(unit 1)
 				)
 				(path "/7204cdda-0a14-40c0-9dc8-8318dd514140/52c3f184-8bc1-44eb-b8c6-96aced11b042/0a77984b-0e61-43a3-838f-8583936efe88"
-					(reference "J50")
+					(reference "J28a")
 					(unit 1)
 				)
 				(path "/7204cdda-0a14-40c0-9dc8-8318dd514140/52c3f184-8bc1-44eb-b8c6-96aced11b042/316b265e-96e5-4e12-ba62-f527eb037ccf"
-					(reference "J51")
+					(reference "J25a")
 					(unit 1)
 				)
 				(path "/7204cdda-0a14-40c0-9dc8-8318dd514140/52c3f184-8bc1-44eb-b8c6-96aced11b042/a5941889-9e91-48ac-996e-3109bbfd970a"
-					(reference "J52")
+					(reference "J26a")
 					(unit 1)
 				)
 				(path "/7204cdda-0a14-40c0-9dc8-8318dd514140/52c3f184-8bc1-44eb-b8c6-96aced11b042/a6f8974c-4bb2-46a6-a2f5-229d9d791f49"
-					(reference "J49")
+					(reference "J27a")
 					(unit 1)
 				)
 				(path "/7204cdda-0a14-40c0-9dc8-8318dd514140/927ab7ec-3c4f-4246-9f54-2bb209e4624c/0a77984b-0e61-43a3-838f-8583936efe88"
-					(reference "J18")
+					(reference "J12a")
 					(unit 1)
 				)
 				(path "/7204cdda-0a14-40c0-9dc8-8318dd514140/927ab7ec-3c4f-4246-9f54-2bb209e4624c/316b265e-96e5-4e12-ba62-f527eb037ccf"
-					(reference "J19")
+					(reference "J9a")
 					(unit 1)
 				)
 				(path "/7204cdda-0a14-40c0-9dc8-8318dd514140/927ab7ec-3c4f-4246-9f54-2bb209e4624c/a5941889-9e91-48ac-996e-3109bbfd970a"
-					(reference "J20")
+					(reference "J10a")
 					(unit 1)
 				)
 				(path "/7204cdda-0a14-40c0-9dc8-8318dd514140/927ab7ec-3c4f-4246-9f54-2bb209e4624c/a6f8974c-4bb2-46a6-a2f5-229d9d791f49"
-					(reference "J17")
+					(reference "J11a")
 					(unit 1)
 				)
 				(path "/7204cdda-0a14-40c0-9dc8-8318dd514140/aa0ac7b6-f653-4dea-a515-ea9099788982/0a77984b-0e61-43a3-838f-8583936efe88"
-					(reference "J12")
+					(reference "J4a")
 					(unit 1)
 				)
 				(path "/7204cdda-0a14-40c0-9dc8-8318dd514140/aa0ac7b6-f653-4dea-a515-ea9099788982/316b265e-96e5-4e12-ba62-f527eb037ccf"
-					(reference "J9")
+					(reference "J1a")
 					(unit 1)
 				)
 				(path "/7204cdda-0a14-40c0-9dc8-8318dd514140/aa0ac7b6-f653-4dea-a515-ea9099788982/a5941889-9e91-48ac-996e-3109bbfd970a"
-					(reference "J10")
+					(reference "J2a")
 					(unit 1)
 				)
 				(path "/7204cdda-0a14-40c0-9dc8-8318dd514140/aa0ac7b6-f653-4dea-a515-ea9099788982/a6f8974c-4bb2-46a6-a2f5-229d9d791f49"
-					(reference "J11")
+					(reference "J3a")
 					(unit 1)
 				)
 				(path "/7204cdda-0a14-40c0-9dc8-8318dd514140/dd925ece-f28f-41db-b9c1-bff66f45860b/0a77984b-0e61-43a3-838f-8583936efe88"
-					(reference "J58")
+					(reference "J32a")
 					(unit 1)
 				)
 				(path "/7204cdda-0a14-40c0-9dc8-8318dd514140/dd925ece-f28f-41db-b9c1-bff66f45860b/316b265e-96e5-4e12-ba62-f527eb037ccf"
-					(reference "J59")
+					(reference "J29a")
 					(unit 1)
 				)
 				(path "/7204cdda-0a14-40c0-9dc8-8318dd514140/dd925ece-f28f-41db-b9c1-bff66f45860b/a5941889-9e91-48ac-996e-3109bbfd970a"
-					(reference "J60")
+					(reference "J30a")
 					(unit 1)
 				)
 				(path "/7204cdda-0a14-40c0-9dc8-8318dd514140/dd925ece-f28f-41db-b9c1-bff66f45860b/a6f8974c-4bb2-46a6-a2f5-229d9d791f49"
-					(reference "J57")
+					(reference "J31a")
 					(unit 1)
 				)
 				(path "/7204cdda-0a14-40c0-9dc8-8318dd514140/e6e426e4-7a0d-4163-9232-4df40c3df7f3/0a77984b-0e61-43a3-838f-8583936efe88"
-					(reference "J34")
+					(reference "J20a")
 					(unit 1)
 				)
 				(path "/7204cdda-0a14-40c0-9dc8-8318dd514140/e6e426e4-7a0d-4163-9232-4df40c3df7f3/316b265e-96e5-4e12-ba62-f527eb037ccf"
-					(reference "J35")
+					(reference "J17a")
 					(unit 1)
 				)
 				(path "/7204cdda-0a14-40c0-9dc8-8318dd514140/e6e426e4-7a0d-4163-9232-4df40c3df7f3/a5941889-9e91-48ac-996e-3109bbfd970a"
-					(reference "J36")
+					(reference "J18a")
 					(unit 1)
 				)
 				(path "/7204cdda-0a14-40c0-9dc8-8318dd514140/e6e426e4-7a0d-4163-9232-4df40c3df7f3/a6f8974c-4bb2-46a6-a2f5-229d9d791f49"
-					(reference "J33")
+					(reference "J19a")
 					(unit 1)
 				)
 				(path "/7204cdda-0a14-40c0-9dc8-8318dd514140/f06dbf80-fe43-424c-832c-ab6085f2b4a7/0a77984b-0e61-43a3-838f-8583936efe88"
-					(reference "J26")
+					(reference "J16a")
 					(unit 1)
 				)
 				(path "/7204cdda-0a14-40c0-9dc8-8318dd514140/f06dbf80-fe43-424c-832c-ab6085f2b4a7/316b265e-96e5-4e12-ba62-f527eb037ccf"
-					(reference "J27")
+					(reference "J13a")
 					(unit 1)
 				)
 				(path "/7204cdda-0a14-40c0-9dc8-8318dd514140/f06dbf80-fe43-424c-832c-ab6085f2b4a7/a5941889-9e91-48ac-996e-3109bbfd970a"
-					(reference "J28")
+					(reference "J14a")
 					(unit 1)
 				)
 				(path "/7204cdda-0a14-40c0-9dc8-8318dd514140/f06dbf80-fe43-424c-832c-ab6085f2b4a7/a6f8974c-4bb2-46a6-a2f5-229d9d791f49"
-					(reference "J25")
+					(reference "J15a")
 					(unit 1)
 				)
 				(path "/7204cdda-0a14-40c0-9dc8-8318dd514140/fb00f2ef-3738-4a3d-8e91-38115c904ed5/0a77984b-0e61-43a3-838f-8583936efe88"
-					(reference "J2")
+					(reference "J8a")
 					(unit 1)
 				)
 				(path "/7204cdda-0a14-40c0-9dc8-8318dd514140/fb00f2ef-3738-4a3d-8e91-38115c904ed5/316b265e-96e5-4e12-ba62-f527eb037ccf"
-					(reference "J3")
+					(reference "J5a")
 					(unit 1)
 				)
 				(path "/7204cdda-0a14-40c0-9dc8-8318dd514140/fb00f2ef-3738-4a3d-8e91-38115c904ed5/a5941889-9e91-48ac-996e-3109bbfd970a"
-					(reference "J4")
+					(reference "J6a")
 					(unit 1)
 				)
 				(path "/7204cdda-0a14-40c0-9dc8-8318dd514140/fb00f2ef-3738-4a3d-8e91-38115c904ed5/a6f8974c-4bb2-46a6-a2f5-229d9d791f49"
-					(reference "J1")
-					(unit 1)
-				)
+					(reference "J7a")
+					(unit 1)
+				)

Commit message: one MCP23017 added and routed
Parts:
- renumbered J7a to J1_07

Commit message: wip
Connections:
- net R13: now also J1_07.78 (Pin_78), J1_07.79 (Pin_79); no longer J1_07.50 (Pin_50), J1_07.51 (Pin_51)
- net R14: now also J1_07.74 (Pin_74), J1_07.75 (Pin_75); no longer J1_07.54 (Pin_54), J1_07.55 (Pin_55)
- net R15: now also J1_07.70 (Pin_70), J1_07.71 (Pin_71); no longer J1_07.58 (Pin_58), J1_07.59 (Pin_59)
- net R16: now also J1_07.66 (Pin_66), J1_07.67 (Pin_67); no longer J1_07.62 (Pin_62), J1_07.63 (Pin_63)
- net R17: now also J1_07.62 (Pin_62), J1_07.63 (Pin_63); no longer J1_07.66 (Pin_66), J1_07.67 (Pin_67)
- net R18: now also J1_07.58 (Pin_58), J1_07.59 (Pin_59); no longer J1_07.70 (Pin_70), J1_07.71 (Pin_71)
- net R19: now also J1_07.54 (Pin_54), J1_07.55 (Pin_55); no longer J1_07.74 (Pin_74), J1_07.75 (Pin_75)
- net R20: now also J1_07.50 (Pin_50), J1_07.51 (Pin_51); no longer J1_07.78 (Pin_78), J1_07.79 (Pin_79)
- net R1 renamed R32
- net R10 renamed R23
- net R11 renamed R22
- net R12 renamed R21
- net R2 renamed R31
- net R3 renamed R30
- net R4 renamed R29
- net R5 renamed R28
- net R6 renamed R27
- net R7 renamed R26
- net R8 renamed R25
- net R9 renamed R24
